Commit message: Assro

File: description/camera.xacro (robot description, xacro)
@@ -4,5 +4,5 @@
         <parent link="chassis"/>
         <child link="camera_link"/>
-        <origin xyz="0.305 0 0.08" rpy="0 0 0"/>
+        <origin xyz="0.048 0 0.142" rpy="0 0 0"/>
     </joint>
     <link name="camera_link">
@@ -11,5 +11,5 @@
                 <box size="0.010 0.03 0.03"/>
             </geometry>
-            <material name="black"/>
+            <material name="red"/>
         </visual>
     </link>

File: description/robot_core.xacro (robot description, xacro)
@@ -6,6 +6,6 @@
     <xacro:property name="chassis_height" value="0.160"/>
     <xacro:property name="chassis_mass" value="2.0"/>
-    <xacro:property name="wheel_radius" value="0.0421"/>
-    <xacro:property name="wheel_thickness" value="0.041"/>
+    <xacro:property name="wheel_radius" value="0.039"/>
+    <xacro:property name="wheel_thickness" value="0.040"/>
     <xacro:property name="wheel_mass" value="0.05"/>
     <xacro:property name="wheel_offset_x" value="0.191"/>
@@ -65,5 +65,5 @@
         <parent link="base_link"/>
         <child link="left_wheel"/>
-        <origin xyz="0 ${wheel_offset_y} 0" rpy="-${pi/2} 0 0" />
+        <origin xyz="0 ${-wheel_offset_y} 0" rpy="-${pi/2} 0 0" />
         <axis xyz="0 0 1"/>
     </joint>
@@ -91,5 +91,5 @@
         <parent link="base_link"/>
         <child link="right_wheel"/>
-        <origin xyz="0 ${-wheel_offset_y} 0" rpy="${pi/2} 0 0" />
+        <origin xyz="0 ${wheel_offset_y} 0" rpy="${pi/2} 0 0" />
         <axis xyz="0 0 -1"/>
     </joint>
