Commit message: ASSRO

File: description/robot_core.xacro (robot description, xacro)
@@ -6,5 +6,5 @@
     <xacro:property name="chassis_height" value="0.160"/>
     <xacro:property name="chassis_mass" value="2.0"/>
-    <xacro:property name="wheel_radius" value="0.0405"/>
+    <xacro:property name="wheel_radius" value="0.042"/>
     <xacro:property name="wheel_thickness" value="0.041"/>
     <xacro:property name="wheel_mass" value="0.05"/>

Commit message: Assro

File: description/robot_core.xacro (robot description, xacro)
@@ -6,5 +6,5 @@
     <xacro:property name="chassis_height" value="0.160"/>
     <xacro:property name="chassis_mass" value="2.0"/>
-    <xacro:property name="wheel_radius" value="0.042"/>
+    <xacro:property name="wheel_radius" value="0.0421"/>
     <xacro:property name="wheel_thickness" value="0.041"/>
     <xacro:property name="wheel_mass" value="0.05"/>

Commit message: tekeryonu

File: description/robot_core.xacro (robot description, xacro)
@@ -73,5 +73,5 @@
         <parent link="base_link"/>
         <child link="left_wheel"/>
-        <origin xyz="0 ${-wheel_offset_y} 0" rpy="-${pi/2} 0 0" />
+        <origin xyz="0 ${wheel_offset_y} 0" rpy="-${pi/2} 0 0" />
         <axis xyz="0 0 1"/>
     </joint>
@@ -99,5 +99,5 @@
         <parent link="base_link"/>
         <child link="right_wheel"/>
-        <origin xyz="0 ${wheel_offset_y} 0" rpy="${pi/2} 0 0" />
+        <origin xyz="0 ${-wheel_offset_y} 0" rpy="${pi/2} 0 0" />
         <axis xyz="0 0 -1"/>
     </joint>
